File: fan.picow.kicad_sch (KiCad schematic)
At the start: 41 parts, among them Q1 BSS138, Q2 BSS138, Q3 IRLML9301, SW1 EG1257, U1 PicoW

Commit message: minor changes
- Change L/C values 300 -> 330
- Change footprint association: 12v pinheader is now vertical
- Change 3D models for capacitors (replaced due to lack of stock)
- Also changed some references to make it more neat
- Add also a square around the fan switch area in the schematic
Other:
- note added: "Fans' Switch"
Changed lines of the file:
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@@
+    (stroke (width 0) (type default) (color 0 0 0 0))
+  )
+  (polyline (pts (xy 95.885 162.56) (xy 19.685 162.56))
     (stroke (width 0) (type default) (color 0 0 0 0))
   )
@@
     (stroke (width 0) (type default) (color 0 0 0 0))
   )
+  (polyline (pts (xy 95.885 106.045) (xy 95.885 162.56))
+    (stroke (width 0) (type default) (color 0 0 0 0))
+  )
   (wire (pts (xy 150.495 127) (xy 150.495 128.905))
     (stroke (width 0) (type default) (color 0 0 0 0))
@@
     (stroke (width 0) (type default) (color 0 0 0 0))
   )
+  (polyline (pts (xy 19.685 106.045) (xy 20.32 106.045))
+    (stroke (width 0) (type default) (color 0 0 0 0))
+  )
   (wire (pts (xy 250.825 33.02) (xy 247.015 33.02))
     (stroke (width 0) (type default) (color 0 0 0 0))
@@
     (stroke (width 0) (type default) (color 0 0 0 0))
   )
+  (polyline (pts (xy 19.685 106.045) (xy 95.885 106.045))
+    (stroke (width 0) (type default) (color 0 0 0 0))
+  )
   (wire (pts (xy 65.405 47.625) (xy 67.31 47.625))
     (stroke (width 0) (type default) (color 0 0 0 0))
@@
     (stroke (width 0) (type default) (color 0 0 0 0))
   )
+  (polyline (pts (xy 19.685 162.56) (xy 19.685 106.045))
+    (stroke (width 0) (type default) (color 0 0 0 0))
+  )
   (polyline (pts (xy 120.015 19.685) (xy 120.015 87.63))
     (stroke (width 0) (type default) (color 0 0 0 0))
@@
   (wire (pts (xy 230.505 155.575) (xy 236.22 155.575))
     (stroke (width 0) (type default) (color 0 0 0 0))
+  )
+  (text "Fans' Switch" (at 20.955 108.585 0)
+    (effects (font (size 1.27 1.27)) (justify left bottom))
   )
   (text "Mounting holes" (at 252.73 125.73 0)
@@
     )
     (path "/86e12817-80ac-414c-aa23-eca04293b568/b8159e12-8a01-4e18-930f-dd9f7045b4ba"
-      (reference "C7") (unit 1) (value "300uF") (footprint "footprints descargados:CAP_EEEFT1V331AP")
+      (reference "C7") (unit 1) (value "330uF") (footprint "footprints descargados:CAP_EEEFT1V331AP")
     )
     (path "/84d2dce4-bf1b-4fde-9c0b-190a062885b2"
@@
     )
     (path "/86e12817-80ac-414c-aa23-eca04293b568/d7641a10-1696-479f-8ad9-c72747f4c20a"
-      (reference "J1") (unit 1) (value "12v Input") (footprint "Connector_PinHeader_2.54mm:PinHeader_1x02_P2.54mm_Horizontal")
+      (reference "J1") (unit 1) (value "12v Input") (footprint "Connector_PinHeader_2.54mm:PinHeader_1x02_P2.54mm_Vertical")
     )
     (path "/86e12817-80ac-414c-aa23-eca04293b568/1790f650-74c6-4ab3-b8d8-2a95be562786"
@@
     )
     (path "/86e12817-80ac-414c-aa23-eca04293b568/53e3d8ec-12b9-4584-97a2-e1df54648bf7"
-      (reference "L1") (unit 1) (value "300uH") (footprint "footprints descargados:DR127-331_INDM125125X800N")
+      (reference "L1") (unit 1) (value "330uH") (footprint "footprints descargados:DR127-331_INDM125125X800N")
     )
     (path "/3fe79dfd-60d0-4881-a73e-44d6645bbde6"
